File: FlightComputer.kicad_sch (KiCad schematic)
At the start: 88 parts, among them J1 B3B-XH-A, J3 DM3D-SF, J4 12401832E402A, U1 AP62150WU-7TSOT26-WU_DIO, U2 TPS2121RUXR, U4 RP2350_60QFN, Y1 ABM8-272-T3

Commit message: fix: derived + added missing vals for passives, cleaned up stuff
Parts:
- C1, C14: value CCHIP-0603(1608-METRIC) -> 10uF
- C10: value CCHIP-0603(1608-METRIC) -> 2.2uF
- C11, C12, C9: value CCHIP-0603(1608-METRIC) -> 0.1uF
- C13: value CCHIP-0603(1608-METRIC) -> 1uF
- C15, C8: value CCHIP-0603(1608-METRIC) -> 100nF
- C16, C17, C18, C20, C21, C22, C23, C24, C25, C27: value CCHIP-0603(1608-METRIC) -> 100n
- C19: value CCHIP-0402(1005-METRIC) -> 100n
- C26, C28, C31: value CCHIP-0603(1608-METRIC) -> 4.7u
- C29, C32: value CCHIP-0402(1005-METRIC) -> 15pF
- C30: value CCHIP-0603(1608-METRIC) -> 1.7u
- C33: value CAPACITORCHIP-0805(2012-METRIC) -> 100nF
- C34: value CCHIP-0603(1608-METRIC) -> 0.47uF
- C35: value CCHIP-0603(1608-METRIC) -> 22uF
- C5, C6: value CAPACITORCHIP-0805(2012-METRIC) -> 0.1u
- C7: value CCHIP-0603(1608-METRIC) -> 10nF
- D2: value CHIP-FLAT-B_0603-0.35MM -> LED
- L1: value INDUCTORCHIP-0805(2012-METRIC) -> 3.3u
- L2: value INDUCTORCHIP-0805(2012-METRIC) -> 3.3uH
- R11: value RESISTOR_CHIP-0805(2012-METRIC) -> 10k
- R12: value RESISTOR_CHIP-0805(2012-METRIC) -> 0k
- R14: value RESISTOR_CHIP-0805(2012-METRIC) -> 1k
- R19: value RCHIP-0603(1608-METRIC) -> 10k
- R3: value RCHIP-0402(1005-METRIC) -> 1k
- R4, R6: value RCHIP-0603(1608-METRIC) -> 1k
- R5: value RCHIP-0603(1608-METRIC) -> 3.3
- R7, R8: value RCHIP-0603(1608-METRIC) -> 27
Connections:
- net +3.3V is gone; now on net +3V3: C6.1, IMU0.5 (VDDIO)
Other:
- note removed: "spi0 debug"
- note removed: "spi1 debug"

Commit message: fixed a loose pin whoops
Connections:
- net at R17.2, R19.1: now also U1.4 (FB)
Changed lines of the file:
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@@
 	)
 	(junction
+		(at 469.9 287.02)
+		(diameter 0)
+		(color 0 0 0 0)
+	)
+	(junction
 		(at 194.31 127)
 		(diameter 0)
@@
 	(wire
 		(pts
-			(xy 469.9 284.48) (xy 469.9 297.18)
+			(xy 469.9 284.48) (xy 469.9 287.02)
 		)
 		(stroke
@@
 	(wire
 		(pts
+			(xy 469.9 287.02) (xy 469.9 297.18)
+		)
+		(stroke
+			(width 0.1524)
+			(type solid)
+		)
+	)
+	(wire
+		(pts
 			(xy 256.54 200.66) (xy 256.54 238.76)
 		)
@@
 	(wire
 		(pts
-			(xy 556.26 287.02) (xy 469.9 287.02)
-		)
-		(stroke
-			(width 0.1524)
-			(type solid)
-		)
-	)
-	(wire
-		(pts
 			(xy 142.24 168.91) (xy 142.24 167.64)
 		)
@@
 		)
 		(stroke
+			(width 0.1524)
+			(type solid)
+		)
+	)
+	(wire
+		(pts
+			(xy 469.9 287.02) (xy 556.26 287.02)
+		)
+		(stroke

Commit message: Start donut shaped PCB
Parts:
- removed C1: 10uF, FlightComputer:CAPC1608X85, symbol FlightComputer:Capacitor_CCHIP-0603(1608-METRIC)
- removed C35: 22uF, FlightComputer:CAPC1608X85, symbol FlightComputer:Capacitor_CCHIP-0603(1608-METRIC)
- removed C8: 100nF, FlightComputer:CAPC1608X85, symbol FlightComputer:Capacitor_CCHIP-0603(1608-METRIC)
- removed D2: LED, FlightComputer:LEDC1608X35N_FLAT-B, symbol FlightComputer:LED_CHIP-FLAT-B_0603-0.35MM
- removed J1: B3B-XH-A, FlightComputer:B3B-XH-A, symbol FlightComputer:Connector_B3B-XH-A
- removed L2: 3.3uH, FlightComputer:INDC2009X120, symbol FlightComputer:Tinkercad_INDUCTORCHIP-0805(2012-METRIC)
- removed R14: 1k, FlightComputer:RESC2012X65, symbol FlightComputer:Tinkercad_RESISTOR_CHIP-0805(2012-METRIC)
- removed R17: 31.6k, FlightComputer:RESC1608X60, symbol FlightComputer:Resistor_RCHIP-0603(1608-METRIC)
- removed R19: 10k, FlightComputer:RESC1608X60, symbol FlightComputer:Resistor_RCHIP-0603(1608-METRIC)
- removed TP1, TP3: TPB1,27, FlightComputer:B1,27, symbol FlightComputer:testpad_TPB1,27
- removed U1: AP62150WU-7TSOT26-WU_DIO, FlightComputer:TSOT26-WU_DIO, symbol FlightComputer:2026-03-13_04-04-58_Library_AP62150WU-7TSOT26-WU_DIO
- BOOT0, RESET0: FOOTPRINT Button_Switch_SMD:SW_Push_1P1T_NO_Vertical_Wuerth_434133025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 -> (none)
- H1, H2, H3, H4: footprint FlightComputer:MOUNTINGHOLE_MOUNTINGHOLE_2.7MM_M2.5 -> MountingHole:MountingHole_2.7mm_M2.5; FOOTPRINT MountingHole:MountingHole_2.7mm_M2.5 -> (none)
- U4: FOOTPRINT RP2350_60QFN_minimal:RP2350-QFN-60-1EP_7x7_P0.4mm_EP3.4x3.4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 -> (none)
- Y1: footprint FlightComputer:CRYSTAL_CRYSTAL_SMD_3225-4PIN_3.2X2.5MM -> Crystal:Crystal_SMD_3225-4Pin_3.2x2.5mm; FOOTPRINT Crystal:Crystal_SMD_3225-4Pin_3.2x2.5mm -> (none)
